File: src/x49_dash/x49_dash.sch (EAGLE design)
At the start: 65 parts, among them J1 1-776276-1, Q1 BSS138, U2 MCP2562

Commit message: x49_dash: WIP total relayout
Parts:
- added U3: (no value), microbuilder:HT16K33_SOP28
- R4, R5: device ngspice-simulation:R -> eagle-ltspice:R
Connections:
- net LEVEL-SHIFT renamed LED_DI_3V3
- net N$52 renamed LED_DI_5V
- net A-2: now also U3.ROW0/A2; no longer U5.ROW8/K6
- net B-2: now also U3.ROW1/A1; no longer U5.ROW9/K7
- net C-2: now also U3.ROW2/A0; no longer U5.ROW10/K8
- net D-2: now also U3.ROW3/K1; no longer U5.ROW11/K9
- net DIG2-1: now also U3.COM0/AD; no longer U5.COM4
- net DIG2-2: now also U3.COM1/KS0; no longer U5.COM5
- net DIG2-3: now also U3.COM2/KS1; no longer U5.COM6
- net DIG2-4: now also U3.COM3/KS2; no longer U5.COM7
- net DP-2: now also U3.ROW7/K5; no longer U5.ROW15/K13/INT
- net E-2: now also U3.ROW4/K2; no longer U5.ROW12/K10
- net F-2: now also U3.ROW5/K3; no longer U5.ROW13/K11
- net G-2: now also U3.ROW6/K4; no longer U5.ROW14/K12
- net GND: now also U3.VSS
- net SCK: now also U3.SCL
- net SDA: now also U3.SDA
- net VIN: now also U3.VDD
Other:
- moved on the sheet: LED3, R4, R5

Commit message: x49_dash: Finish relayout
Parts:
- removed LCD1: LCD-16X2NOHOLES, SparkFun-Displays:LCD-16X2NOHOLES
- removed R7: 10k, rcl:POTENTIOMETER_PT-10S
- U1: value (none) -> +12v; device SparkFun-IC-Power:V_REG_78XX-TO-220 -> SparkFun-IC-Power:V_REG_78XX7812
Connections:
- removed net LCD-D0: LCD1.DB0, U$1.7/RX3
- removed net LCD-D1: LCD1.DB1, U$1.8/TX3
- removed net LCD-D2: LCD1.DB2, U$1.9/RX2/PWM
- removed net LCD-D3: LCD1.DB3, U$1.21/A7/PWM
- removed net LCD-D4: LCD1.DB4, U$1.14/A1
- removed net LCD-D5: LCD1.DB5, U$1.15/A1/T
- removed net LCD-D6: LCD1.DB6, U$1.16/A2/T
- removed net LCD-D7: LCD1.DB7, U$1.17/A3/T
- removed net LCD-E: LCD1.E, U$1.20/A6/PWM
- removed net LCD-RS: LCD1.RS, U$1.19/A5/T/SCL0
- removed net N$27: LCD1.VO, R7.3
- net GND: no longer LCD1.R/W, LCD1.VSS, R7.1
- net VIN: no longer LCD1.VDD, R7.2

Commit message: x49_dash: Rev 1B
Parts:
- added R11, R14, R6, R7: 10k, eagle-ltspice:R
- added S1, S2, S5, S6: MOMENTARY-SWITCH-SPST-SMD-12MM, SparkFun-Switches:MOMENTARY-SWITCH-SPST-SMD-12MM
- added U$2: ADAFRUIT-OLED-BREAKOUT, adafruit:ADAFRUIT-OLED-BREAKOUT
Connections:
- removed net 3.3V: Q1.G, R12.2, U2.VIO
- new net BUTTON-2: R7.1, S2.2, U$1.21/A7/PWM
- new net BUTTON-3: R11.1, S3.2, U$1.22/A8/T/PWM
- new net BUTTON-4: R14.1, S4.2, U$1.23/A9/T/PWM
- new net BUTTON-5: R3.1, S5.2, U$1.5/PWM
- new net MISO: U$1.12/MISO, U$2.MISO
- new net MOSI: U$1.11/MOSI, U$2.MOSI
- new net OLED_CS: U$1.10/TX2/PWM, U$2.OLED_CS
- new net OLED_DC: U$1.15/A1/T, U$2.OLED_DC
- new net OLED_RESET: U$1.14/A1, U$2.RESET
- new net SCL: R5.1, U$1.19/A5/T/SCL0, U3.SCL, U5.SCL
- new net SDCARD_CD: U$1.8/TX3, U$2.SDCARD_CD
- new net SDCARD_CS: U$1.9/RX2/PWM, U$2.SDCARD_CS
- new net VDD_3V3: Q1.G, R11.2, R12.2, R14.2, R6.2, R7.2, U$1.3.3V, U2.VIO
- net BUTTON-1: now also R6.1, S1.2, U$1.20/A6/PWM; no longer R3.1, S4.2, U$1.5/PWM
- net FLEX: now also S6.2; no longer S3.2
- net GND: now also S1.1, S2.1, S5.1, S6.1, U$2.GND
- net LED_DI_3V3: now also U$1.2; no longer U$1.22/A8/T/PWM
- net SCK: now also U$2.CLK; no longer R5.1, U3.SCL, U5.SCL
- net VIN: now also U$2.VIN
Other:
- moved on the sheet: H1, H2, H3, H4, R5, S3, S4
