File: src/x50_daq_wheelboardrear/wheel_board_rear.sch (EAGLE design)
At the start: 34 parts, among them J1 1-776087-1, J3 DTF13-4P, U1 PCA9518PWRSOIC-20, U2 LM1117, U3 LM1117

Commit message: Add files via upload
Connections:
- removed net N$11: J1.11, R1.2
- removed net N$15: J1.14, R3.2
- new net N$6: J1.19, R1.2
- new net N$7: J1.22, R3.2
- net 2.6V: now also J1.13, J1.9
- net EXT_SCL1: now also J1.3
- net EXT_SCL2: now also J1.7
- net EXT_SCL3: now also J1.11
- net EXT_SCL4: now also J1.15
- net EXT_SDA1: now also J1.4
- net EXT_SDA2: now also J1.8
- net EXT_SDA3: now also J1.12
- net EXT_SDA4: now also J1.16
- net GND: now also J1.14, J1.18, J1.21; no longer J1.13
- net SCL0: no longer J1.3
- net SCL1: no longer J1.7
- net SDA0: no longer J1.4
- net SDA1: no longer J1.8
- net VIN: now also J1.17, J1.20; no longer J1.12, J1.9
Other:
- moved on the sheet: R1, R2, R3, R5
