File: src/x50_daq_wheelboardrear/wheel_board_rear.brd (EAGLE design)
At the start: 66.3 x 73 mm, 34 parts, among them J1 1-776087-1, J3 DTF13-4P, U1 PCA9518PWRSOIC-20, U2 LM1117, U3 LM1117

Commit message: Add files via upload
Connections:
- removed net N$11: J1.11, R1.2
- removed net N$15: J1.14, R3.2
- new net N$6: J1.19, R1.2
- new net N$7: J1.22, R3.2
- net 2.6V: now also J1.13, J1.9
- net EXT_SCL1: now also J1.3
- net EXT_SCL2: now also J1.7
- net EXT_SCL3: now also J1.11
- net EXT_SCL4: now also J1.15
- net EXT_SDA1: now also J1.4
- net EXT_SDA2: now also J1.8
- net EXT_SDA3: now also J1.12
- net EXT_SDA4: now also J1.16
- net GND: now also J1.14, J1.18, J1.21; no longer J1.13
- net SCL0: no longer J1.3
- net SCL1: no longer J1.7
- net SDA0: no longer J1.4
- net SDA1: no longer J1.8
- net VIN: now also J1.17, J1.20; no longer J1.12, J1.9
Routing:
- net EXT_SDA1: track 4.76 -> 90.0 mm
- net EXT_SCL2: track 4.77 -> 88.1 mm
- net SDA0: track 106.0 -> 34.8 mm, vias 0 -> 1
- net SCL0: track 103.9 -> 41.1 mm, vias 2 -> 1
- net EXT_SDA4: track 3.61 -> 64.0 mm
- net SDA1: track 58.9 -> 0.00 mm
- net EXT_SDA2: track 8.62 -> 66.1 mm
- net SCL1: track 47.7 -> 0.00 mm
- net EXT_SCL1: track 3.93 -> 49.1 mm, vias 0 -> 2
- net 2.6V: track 123.4 -> 162.6 mm, vias 1 -> 0
- net EXT_SCL3: track 8.41 -> 41.2 mm, vias 1 -> 2
- net EXT_SCL4: track 4.13 -> 36.0 mm, vias 0 -> 1
- net EXT_SDA3: track 4.13 -> 35.2 mm, vias 0 -> 1
- net N$7: track 0.00 -> 19.0 mm
- net N$6: track 0.00 -> 18.4 mm
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
Commit message: Add files via upload
Parts:
- moved R7 2.03 mm to (69.4, 60.1), turned to 90 degrees
- moved R8 1.59 mm to (68.9, 37.8)
- moved R9 1.59 mm to (66.4, 37.8)
- moved J3 1.59 mm to (44.7, 73.9)
- moved R12 1.59 mm to (56.2, 37.8)
- moved R13 1.59 mm to (61.3, 37.8)
- moved R16 1.59 mm to (58.7, 37.8)
- moved U$1 1.59 mm to (29.2, 61.7)
- moved C2 1.59 mm to (40.9, 40.2)
- moved R10 1.59 mm to (63.8, 59.8)
- moved R11 1.59 mm to (58.7, 59.8)
- moved R14 1.59 mm to (61.2, 59.8)
- moved R15 1.59 mm to (56.2, 59.8)
- moved R19 1.59 mm to (33.3, 42.8)
- moved R21 1.59 mm to (38.4, 33.9)
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Routing:
- net EXT_SCL2: track 88.1 -> 75.7 mm
- net 2.6V: track 162.6 -> 151.8 mm
- net N$3: track 11.1 -> 3.37 mm
- net SCL0: track 41.1 -> 38.4 mm
- net A1: track 55.8 -> 54.3 mm
- net EN4: track 30.6 -> 31.7 mm
- net EXT_SCL4: track 36.0 -> 35.3 mm
- net EXT_SDA2: track 66.1 -> 65.5 mm
