File: src/x50_daq_wheelboardfront/wheel_board_front.brd (EAGLE design)
At the start: 73.6 x 94.9 mm, 33 parts, among them IC1 LM2903D, IC2 74HC590D, IC3 74HC590D, IC4 74HC590D, IC5 4098D, IC6 MCP23017SO, IC7 MCP23017SO, IC8 OV-0100-C7OV-0100-C7, J1 1-776087-1, J3 DTF13-4P, U1 SN74HC573ADW, U2 LM1117, U3 SN74HC573ADW, U4 SN74HC573ADW

Commit message: Add files via upload
Connections:
- removed net VDD12V_BOARD: J3.1
- new net SCL1: J1.10, U$3.D16/A2
- new net SDA1: J1.11, U$3.D17/A3
- net SCL0: no longer J1.10
- net SDA0: no longer J1.11
- net VIN: now also J3.1
Routing:
- net SCL1: track 0.00 -> 80.5 mm, vias 0 -> 6
- net SDA1: track 0.00 -> 79.8 mm, vias 0 -> 5
- net SCL0: track 135.5 -> 121.0 mm
- net SDA0: track 139.2 -> 127.2 mm
- net VIN: track 373.1 -> 380.2 mm
- net N$2: track 62.6 -> 65.4 mm
