File: src/x50_daq_wheelboardfront/wheel_board_front.sch (EAGLE design)
At the start: 33 parts, among them IC1 LM2903D, IC2 74HC590D, IC3 74HC590D, IC4 74HC590D, IC5 4098D, IC6 MCP23017SO, IC7 MCP23017SO, IC8 OV-0100-C7OV-0100-C7, J1 1-776087-1, J3 DTF13-4P, U1 SN74HC573ADW, U2 LM1117, U3 SN74HC573ADW, U4 SN74HC573ADW

Commit message: Add files via upload
Connections:
- removed net VDD12V_BOARD: J3.1
- new net SCL1: J1.10, U$3.D16/A2
- new net SDA1: J1.11, U$3.D17/A3
- net SCL0: no longer J1.10
- net SDA0: no longer J1.11
- net VIN: now also J3.1
Changed lines of the file:
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@@
 </busses>
 <nets>
-<net name="VDD12V_BOARD" class="0">
-<segment>
-<pinref part="J3" gate="G$1" pin="1"/>
-<wire x1="129.54" y1="78.74" x2="116.84" y2="78.74" width="0.1524" layer="91"/>
-<label x="109.22" y="78.74" size="1.778" layer="95"/>
-</segment>
-</net>
 <net name="GND" class="1">
 <segment>
@@
 <wire x1="55.88" y1="86.36" x2="55.88" y2="88.9" width="0.1524" layer="91"/>
 <label x="55.88" y="88.9" size="1.778" layer="95"/>
+</segment>
+<segment>
+<pinref part="J3" gate="G$1" pin="1"/>
+<wire x1="129.54" y1="78.74" x2="116.84" y2="78.74" width="0.1524" layer="91"/>
+<label x="116.84" y="78.74" size="1.778" layer="95"/>
 </segment>
 </net>
@@
 </segment>
 <segment>
-<pinref part="J1" gate="G$1" pin="11"/>
-<wire x1="132.08" y1="20.32" x2="124.46" y2="20.32" width="0.1524" layer="91"/>
-<label x="124.46" y="20.32" size="1.778" layer="95"/>
-</segment>
-<segment>
 <pinref part="IC7" gate="G$1" pin="SDA"/>
 <wire x1="-88.9" y1="-63.5" x2="-93.98" y2="-63.5" width="0.1524" layer="91"/>
@@
 <wire x1="132.08" y1="35.56" x2="124.46" y2="35.56" width="0.1524" layer="91"/>
 <label x="124.46" y="35.56" size="1.778" layer="95"/>
-</segment>
-<segment>
-<pinref part="J1" gate="G$1" pin="10"/>
-<wire x1="132.08" y1="22.86" x2="124.46" y2="22.86" width="0.1524" layer="91"/>
-<label x="124.46" y="22.86" size="1.778" layer="95"/>
 </segment>
 <segment>
@@
 </segment>
 </net>
+<net name="SDA1" class="0">
+<segment>
+<pinref part="U$3" gate="G$1" pin="D17/A3"/>
+<wire x1="-139.7" y1="27.94" x2="-130.81" y2="27.94" width="0.1524" layer="91"/>
+<label x="-133.35" y="27.94" size="1.778" layer="95"/>
+</segment>
+<segment>
+<pinref part="J1" gate="G$1" pin="11"/>
+<wire x1="132.08" y1="20.32" x2="124.46" y2="20.32" width="0.1524" layer="91"/>
+<label x="124.46" y="20.32" size="1.778" layer="95"/>
+</segment>
+</net>
+<net name="SCL1" class="0">
+<segment>
+<pinref part="U$3" gate="G$1" pin="D16/A2"/>
+<wire x1="-139.7" y1="24.13" x2="-130.81" y2="24.13" width="0.1524" layer="91"/>
+<label x="-133.35" y="24.13" size="1.778" layer="95"/>
+</segment>
+<segment>
+<pinref part="J1" gate="G$1" pin="10"/>
+<wire x1="132.08" y1="22.86" x2="124.46" y2="22.86" width="0.1524" layer="91"/>
+<label x="124.46" y="22.86" size="1.778" layer="95"/>
+</segment>
+</net>
